Commit message: feat(model): the fixture, and the telescope, take the C3 fit
Regenerate test/description/pzs100.urdf from the live xacro: fitted damping on
all five axes, Coulomb to zero on slew and telescope, gripper limits 0.2/0.7/0.5
to 0.0/0.538/0.12. It was a 2026-08-31 snapshot and crane_mpc bakes its solver
from it, so the shipped solver carried the pre-fit plant.

Empty damping_overrides. Its one row forced the telescope to 0.0 because no
identified value existed; the C3 fit gives 5.640e4 and Marc's stack an
independent 5.94e4.

Guard the snapshot, which --check cannot: test_description_snapshot re-expands
the description with the launch file's own arguments and diffs. It fails rather
than skips when the description is not on the index.

allowed_collisions.srdf and collision_model.hpp re-derived - the gripper limits
move four reasons, the pair set is unchanged.

File: test/description/pzs100.urdf (robot description, URDF)
Before this commit: robot crane_model, 49 links, 48 joints
Joints:
- joint q11_right_rail_joint: limit lower=0.2 upper=0.7 effort=1e4 velocity=0.5 -> lower=0.0 upper=0.538 effort=1e4 velocity=0.12
- joint q9_left_rail_joint: limit lower=0.2 upper=0.7 effort=1e4 velocity=0.5 -> lower=0.0 upper=0.538 effort=1e4 velocity=0.12

Commit message: 126-cylinder-ratio-sign-and-poles: The arm's transmission ratio changes sign inside its own box, and the row divides by it

File: test/description/pzs100.urdf (robot description, URDF)
Before this commit: robot crane_model, 49 links, 48 joints
Links:
- removed link K1_boom_cylinder_suspension
- removed link K2_arm_cylinder_suspension
- added link K1_boom_cylinder_linkage_big_mounting_on_slewing_column
- added link K1_boom_cylinder_mounting_on_slewing_column
- added link K2_arm_cylinder_left_suspension
- added link K2_arm_cylinder_right_suspension
- added link K2_boom_cylinder_linkage_small_mounting_on_boom
- added link K3_arm_cylinder_piston_left_suspension
- added link K3_arm_cylinder_piston_right_suspension
Joints:
- removed joint K1_boom_cylinder_suspension_fix
- removed joint K2_arm_cylinder_suspension_fix
- added joint arm_cylinder_left_suspension_fix: type fixed, parent K2_boom, child K2_arm_cylinder_left_suspension, origin xyz=-1.6802 -0.0485 -0.224 rpy=0 0 0
- added joint arm_cylinder_piston_left_suspension_fix: type fixed, parent K3_arm, child K3_arm_cylinder_piston_left_suspension, origin xyz=0.274489018947000 -0.224000000000000 0.468000481872000 rpy=0 0 0
- added joint arm_cylinder_piston_right_suspension_fix: type fixed, parent K3_arm, child K3_arm_cylinder_piston_right_suspension, origin xyz=0.274489018947000 0.224000000000000 0.468000481872000 rpy=0 0 0
- added joint arm_cylinder_right_suspension_fix: type fixed, parent K2_boom, child K2_arm_cylinder_right_suspension, origin xyz=-1.6802 -0.0485 0.224 rpy=0 0 0
- added joint boom_cylinder_linkage_big_mounting_on_slewing_column_fix: type fixed, parent K1_slewing_column, child K1_boom_cylinder_linkage_big_mounting_on_slewing_column, origin xyz=-0.120000 -0.070000 0 rpy=0 0 0
- added joint boom_cylinder_linkage_small_mounting_on_boom_fix: type fixed, parent K2_boom, child K2_boom_cylinder_linkage_small_mounting_on_boom, origin xyz=-3.039426 -0.036293 0 rpy=0 0 0
- added joint boom_cylinder_mounting_on_slewing_column_fix: type fixed, parent K1_slewing_column, child K1_boom_cylinder_mounting_on_slewing_column, origin xyz=0.433000 -1.774000 0 rpy=0 0 0
